File: Controller/PCB/controller/controller.kicad_sch (KiCad schematic)
At the start: 75 parts, among them Q1 S9013, Q2 S9013, Q3 S9013, Q4 S9013, Q5 S9013, SW1 SW_SPDT, SW2 SW_SPDT, U1 Joystick, U2 Joystick, U3 NLAS4684, U4 NLAS4684, U5 LM2940-5.0

Commit message: Update Schematic and Continue to work on Cpp
Parts:
- removed J?: SERIAL_DEBUG_CONNECTOR, symbol Connector_Generic:Conn_02x06_Odd_Even
- added C10: 10uF, symbol Device:C
- added D9: RED, LED_SMD:LED_0603_1608Metric, symbol Device:LED
- added J2: SERIAL_DEBUG_Conn, Connector_PinHeader_2.54mm:PinHeader_2x04_P2.54mm_Vertical_SMD, symbol Connector_Generic:Conn_02x04_Odd_Even
- added Q6: S9013, Package_TO_SOT_SMD:SOT-23, symbol Transistor_BJT:2N2219
- added R34: 4K7, Resistor_SMD:R_0603_1608Metric, symbol Device:R
- added R35: 1K, Resistor_SMD:R_0603_1608Metric, symbol Device:R
- D1, D4: value LED -> RED
- D2, D5, D7, D8: value LED -> BLUE
- D3: value LED -> GREEN
- J1: renamed from J?; footprint (none) -> Connector_PinHeader_2.54mm:PinHeader_2x04_P2.54mm_Vertical_SMD
- POT_1, POT_2: footprint (none) -> My_library:PDB12 Series
- R25, R31, R33: value 1K -> 390R
- R27, R29: value 1K -> 2K
- renumbered Btn_5 to RESET1
Connections:
- net +3V3: now also J2.2 (Pin_2), J2.7 (Pin_7)
- net +5V: now also C10.1, D9.2 (A)
- net DEBUG: now also J2.1 (Pin_1)
- net DEBUG_IRQ: now also J2.6 (Pin_6)
- net DEBUG_MISO: now also J2.5 (Pin_5)
- net DEBUG_MOSI: now also J2.4 (Pin_4)
- net Earth: now also C9.2, C10.2, Q6.1 (E)
- net NRF_SCK: now also J2.3 (Pin_3)
- new net: D9.1 (K), R35.2
- new net: Q6.3 (C), R35.1
- new net: Q6.2 (B), R34.1
- new net DEBUG_WRONG_WAY: J2.8 (Pin_8), R34.2
Other:
- moved on the sheet: C9

Commit message: Updates
Connections:
- net +5V: now also SW2.1 (A)
Changed lines of the file:
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@@
     (pin "1")
   )
-  (symbol (lib_id "power:+5V") (at 157.48 21.59 0) (unit 1)
+  (symbol (lib_id "power:+5V") (at 157.48 20.32 0) (unit 1)
     (in_bom yes) (on_board yes)
-    (property "Reference" "#PWR0148" (id 0) (at 157.48 25.4 0)
+    (property "Reference" "#PWR0148" (id 0) (at 157.48 24.13 0)
       (effects (font (size 1.27 1.27)) hide)
     )
-    (property "Value" "+5V" (id 1) (at 157.861 17.1958 0))
-    (property "Footprint" "" (id 2) (at 157.48 21.59 0)
+    (property "Value" "+5V" (id 1) (at 157.861 15.9258 0))
+    (property "Footprint" "" (id 2) (at 157.48 20.32 0)
       (effects (font (size 1.27 1.27)) hide)
     )
-    (property "Datasheet" "" (id 3) (at 157.48 21.59 0)
+    (property "Datasheet" "" (id 3) (at 157.48 20.32 0)
       (effects (font (size 1.27 1.27)) hide)
     )
