File: Controller/PCB/controller/controller.kicad_pcb (KiCad board)
At the start: 2 copper layers, 106.7 x 99.1 mm, 57 parts, among them J1 nRF24L01_Conn, Q1 S9013, Q2 S9013, Q4 S9013, SW1 SW_SPDT, U1 Joystick, U2 Joystick, U3 LM2940-3.0, U5 LM2940-5.0

Commit message: Finalise PCB Schematic
Parts:
- moved C3 21.8 mm to (128.3, 115.1)
- moved R2 21.8 mm to (130.8, 116.8)
- moved R3 16.6 mm to (119.4, 101.6)
- moved C4 16.3 mm to (116.0, 101.6), turned to 90 degrees
- moved R5 10.9 mm to (185.4, 100.8), turned to 180 degrees
- moved C6 10.9 mm to (187.6, 104.1)
- moved C5 9.09 mm to (182.9, 114.3)
- moved R4 8.59 mm to (181.2, 111.6)
- moved R26 5.52 mm to (170.2, 57.2)
- moved U2 3.81 mm to (194.3, 114.3)
- moved U1 3.81 mm to (115.6, 114.3)
- moved R24 3.80 mm to (175.3, 57.2)
- moved Q2 2.54 mm to (185.4, 132.1)
- moved R10 2.54 mm to (185.4, 142.2)
- moved BT1 2.54 mm to (139.7, 103.6)
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Connections:
- A1 pad 13: SERIAL_MISO -> NRF_MISO
- A1 pad 5: SERIAL_MOSI -> NRF_MOSI
Routing:
- net +5V: track 0.00 -> 322.6 mm
- net +3V3: track 0.00 -> 139.6 mm, vias 0 -> 2
- net SW_1: track 0.00 -> 128.1 mm, vias 0 -> 2
- net BAT_PWR: track 0.00 -> 122.1 mm, vias 0 -> 1
- net LED_1: track 0.00 -> 112.6 mm
- net Net-(BT1-Pad2): track 0.00 -> 97.0 mm
- net RESET: track 0.00 -> 91.1 mm, vias 0 -> 2
- net R_ROLL: track 0.00 -> 80.8 mm, vias 0 -> 2
- net Btn_1: track 0.00 -> 67.3 mm, vias 0 -> 2
- net Btn_3: track 0.00 -> 67.1 mm, vias 0 -> 2
- net +BATT: track 0.00 -> 62.1 mm
- net Btn_2: track 0.00 -> 61.4 mm, vias 0 -> 2
- net NRF_MOSI: track 0.00 -> 45.7 mm, vias 0 -> 2
- net L_ROLL: track 0.00 -> 42.4 mm, vias 0 -> 2
- net R_PITCH: track 0.00 -> 39.5 mm
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- added copper zone on B.Cu, net Earth
- added copper zone on F.Cu, net Earth
Other:
- board size 106.7 x 99.1 mm -> 99.1 x 99.1 mm
