File: Reciever-Main/PCB/Main-Craft-PCB/Main-Craft-PCB/Main-Craft-PCB.kicad_sch (KiCad schematic)
At the start: 126 parts, among them J1 nRF24L01_Conn, J10 L298N, J2 IR_SENSOR_?, J3 IR_SENSOR_?, J4 IR_SENSOR_?, J5 IR_SENSOR_?, J6 ESC_?, J7 ESC_?, J8 ESC_?, J9 ESC_?, Q1 2N2219, Q10 2N2219, Q11 2N2219, Q12 2N2219, Q13 2N2219, Q14 2N2219, Q2 2N2219, Q3 2N2219, Q4 2N2219, Q5 2N2219, Q6 2N2219, Q7 2N2219, Q8 2N2219, Q9 2N2219, SW1 SW_Push, SW2 SW_Push, SW3 SW_Push, SW4 SW_SPDT, SW5 SW_SPDT, SW6 SW_SPDT, SW7 SW_SPDT, SW8 SW_SPDT, U1 NUCLEO144-F429ZI, U2 LM741, U3 LM741, U4 LM2940-3.0, U5 LM2940-5.0, U6 LM2940-12.0

Commit message: START SCHEMATIC
Parts:
- SW4, SW5, SW6, SW7, SW8, U6: footprint (none) -> My_library:KNX-1-D1
- U4, U5: footprint (none) -> Package_TO_SOT_SMD:SOT-223
Changed lines of the file:
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@@
       (effects (font (size 1.27 1.27)) (justify left))
     )
-    (property "Footprint" "" (id 2) (at 238.76 96.52 0)
+    (property "Footprint" "My_library:KNX-1-D1" (id 2) (at 238.76 96.52 0)
       (effects (font (size 1.27 1.27)) hide)
     )
@@
       (effects (font (size 1.27 1.27)) (justify left))
     )
-    (property "Footprint" "" (id 2) (at 267.97 96.52 0)
+    (property "Footprint" "My_library:KNX-1-D1" (id 2) (at 267.97 96.52 0)
       (effects (font (size 1.27 1.27)) hide)
     )
@@
     (property "Reference" "U5" (id 0) (at 375.92 186.69 0))
     (property "Value" "LM2940-5.0" (id 1) (at 375.92 189.23 0))
-    (property "Footprint" "" (id 2) (at 375.92 194.31 0)
+    (property "Footprint" "Package_TO_SOT_SMD:SOT-223" (id 2) (at 375.92 194.31 0)
       (effects (font (size 1.27 1.27)) hide)
     )
@@
       (effects (font (size 1.27 1.27)) (justify left))
     )
-    (property "Footprint" "" (id 2) (at 256.54 62.23 0)
+    (property "Footprint" "My_library:KNX-1-D1" (id 2) (at 256.54 62.23 0)
       (effects (font (size 1.27 1.27)) hide)
     )
@@
     (property "Reference" "U4" (id 0) (at 375.92 163.83 0))
     (property "Value" "LM2940-3.0" (id 1) (at 375.92 166.37 0))
-    (property "Footprint" "" (id 2) (at 375.92 171.45 0)
+    (property "Footprint" "Package_TO_SOT_SMD:SOT-223" (id 2) (at 375.92 171.45 0)
       (effects (font (size 1.27 1.27)) hide)
     )
@@
       (effects (font (size 1.27 1.27)) (justify right))
     )
-    (property "Footprint" "" (id 2) (at 379.73 74.93 0)
+    (property "Footprint" "My_library:KNX-1-D1" (id 2) (at 379.73 74.93 0)
       (effects (font (size 1.27 1.27)) hide)
     )
@@
     (property "Reference" "U6" (id 0) (at 375.92 210.82 0))
     (property "Value" "LM2940-12.0" (id 1) (at 375.92 213.36 0))
-    (property "Footprint" "" (id 2) (at 375.92 218.44 0)
+    (property "Footprint" "My_library:KNX-1-D1" (id 2) (at 375.92 218.44 0)
       (effects (font (size 1.27 1.27)) hide)
     )
@@
       (effects (font (size 1.27 1.27)) (justify left))
     )
-    (property "Footprint" "" (id 2) (at 280.67 62.23 0)
+    (property "Footprint" "My_library:KNX-1-D1" (id 2) (at 280.67 62.23 0)
       (effects (font (size 1.27 1.27)) hide)
     )
@@
     )
     (path "/2509dca9-2b73-48fa-a5e6-42e0aa1795c8"
-      (reference "SW4") (unit 1) (value "SW_SPDT") (footprint "")
+      (reference "SW4") (unit 1) (value "SW_SPDT") (footprint "My_library:KNX-1-D1")
     )
     (path "/84321168-615d-4561-a7cc-0c639f0b2e66"
-      (reference "SW5") (unit 1) (value "SW_SPDT") (footprint "")
+      (reference "SW5") (unit 1) (value "SW_SPDT") (footprint "My_library:KNX-1-D1")
     )
     (path "/2b04ed5e-be17-4f74-baa7-c28a76ed7f9a"
-      (reference "SW6") (unit 1) (value "SW_SPDT") (footprint "")
+      (reference "SW6") (unit 1) (value "SW_SPDT") (footprint "My_library:KNX-1-D1")
     )
     (path "/efc7374d-56dd-41e1-8589-0105adc72ef6"
-      (reference "SW7") (unit 1) (value "SW_SPDT") (footprint "")
+      (reference "SW7") (unit 1) (value "SW_SPDT") (footprint "My_library:KNX-1-D1")
     )
     (path "/a939a636-0de0-4fa0-bbc3-54587417098d"
-      (reference "SW8") (unit 1) (value "SW_SPDT") (footprint "")
+      (reference "SW8") (unit 1) (value "SW_SPDT") (footprint "My_library:KNX-1-D1")
     )
     (path "/7b448334-a672-4f67-8bb7-9dc7daa7fefe"
@@
     )
     (path "/885e2e55-5c0e-4681-9913-7987da6917ea"
-      (reference "U4") (unit 1) (value "LM2940-3.0") (footprint "")
+      (reference "U4") (unit 1) (value "LM2940-3.0") (footprint "Package_TO_SOT_SMD:SOT-223")
     )
     (path "/61f626fc-a4e9-4e91-a422-6f85daa7effb"
-      (reference "U5") (unit 1) (value "LM2940-5.0") (footprint "")
+      (reference "U5") (unit 1) (value "LM2940-5.0") (footprint "Package_TO_SOT_SMD:SOT-223")
     )
     (path "/b99d1638-b577-4f10-9b67-afeca6a9d8c0"
-      (reference "U6") (unit 1) (value "LM2940-12.0") (footprint "")
+      (reference "U6") (unit 1) (value "LM2940-12.0") (footprint "My_library:KNX-1-D1")
     )
   )
