File: Main-Craft-PCB/Main-Craft-PCB/_autosave-Main-Craft-PCB.kicad_sch (KiCad schematic)
At the start: 88 parts, among them J1 Conn_01x10, Q23 BC817, Q25 IRFR9014PBF, Q31 BC817, U10 ZLDO1117G50TA, U2 NUCLEO144-F429ZI, U5 74HC14, U9 ZSR330GTA

Commit message: add to schematic
Parts:
- added D1, D2, D3, D4, D5, D6, D7: BLUE, LED_SMD:LED_0603_1608Metric, symbol Device:LED
- added Q1, Q2, Q3, Q4, Q5, Q6, Q7: S9013, Package_TO_SOT_SMD:SOT-23, symbol Transistor_BJT:2N2219
- added R1, R3, R5, R7, R? (x3): 4K7, Resistor_SMD:R_0603_1608Metric, symbol Device:R
- added R2, R4, R6, R8, R? (x3): 1K, Resistor_SMD:R_0603_1608Metric, symbol Device:R
Connections:
- net +5V: now also D1.2 (A), D2.2 (A), D3.2 (A), D4.2 (A), D5.2 (A), D6.2 (A), D7.2 (A)
- net Earth: now also Q1.1 (E), Q2.1 (E), Q3.1 (E), Q4.1 (E), Q5.1 (E), Q6.1 (E), Q7.1 (E)
- net LED_1: now also R1.2, R3.2, R5.2, R7.2, R?.2, R?.2, R?.2
- new net: Q3.2 (B), R?.1
- new net: Q3.3 (C), R?.1
- new net: Q2.2 (B), R?.1
- new net: Q5.3 (C), R4.1
- new net: D5.1 (K), R4.2
- new net: Q2.3 (C), R?.1
- new net: D1.1 (K), R?.2
- new net: Q1.2 (B), R?.1
- new net: Q1.3 (C), R?.1
- new net: Q6.2 (B), R5.1
- new net: D2.1 (K), R?.2
- new net: Q5.2 (B), R3.1
- new net: D4.1 (K), R2.2
- new net: Q4.2 (B), R1.1
- new net: Q6.3 (C), R6.1
- new net: D6.1 (K), R6.2
- new net: D3.1 (K), R?.2
- new net: Q7.3 (C), R8.1
- new net: D7.1 (K), R8.2
- new net: Q7.2 (B), R7.1
- new net: Q4.3 (C), R2.1
Other:
- moved on the sheet: D?, Q?, R?
