File: LiDAR-Main/Schematic/LiDAR-Board/LiDAR-Board.kicad_pcb (KiCad board)
At the start: 2 copper layers, 0 parts

Commit message: Connector on schematic
Parts:
- added Q1: NPN, Package_TO_SOT_SMD:SOT-23, F.Cu at (54.9, 27.9)
- added Q2: NPN, Package_TO_SOT_SMD:SOT-23, F.Cu at (54.9, 33.0)
- added R1: 10K, Resistor_SMD:R_0603_1608Metric, F.Cu at (50.8, 27.9)
- added R2: 10K, Resistor_SMD:R_0603_1608Metric, F.Cu at (50.8, 33.0)
- added U1: Pico, HEVCS_Sensor_Footprints:Pi_Pico, F.Cu at (31.9, 49.5)
- added U2: ~, HEVCS_Sensor_Footprints:Conn_01x05_MOLEX, F.Cu at (76.2, 30.5)
- added U3: ~, HEVCS_Sensor_Footprints:Conn_01x05_MOLEX, F.Cu at (76.2, 45.7)
- added U4: ~, HEVCS_Sensor_Footprints:Conn_01x05_MOLEX, F.Cu at (76.2, 61.0)
