File: LiDAR-Main/Schematic/LiDAR-Board/LiDAR-Board.kicad_pcb (KiCad board)
At the start: 2 copper layers, 39.4 x 54.4 mm, 12 parts, among them J1 Conn_01x04, Q1 NPN, Q2 NPN, U1 Pico

Commit message: Corrected Tx/Rx assignment
Connections:
- J1 pad 2: UART_0_TX -> UART_0_RX
- J1 pad 3: UART_0_RX -> UART_0_TX
Routing:
- net UART_0_TX: track 8.65 -> 6.86 mm
- net UART_0_RX: track 6.33 -> 6.96 mm
Changed lines of the file:
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@@
       (outputformat 1)
       (mirror false)
-      (drillshape 1)
+      (drillshape 0)
       (scaleselection 1)
-      (outputdirectory "")
+      (outputdirectory "Gerber_Output/")
     )
   )
@@
       (net 34 "5V_MAIN_BOARD") (pinfunction "Pin_1") (pintype "passive"))
     (pad "2" thru_hole circle (at -1.524 0 90) (size 1.524 1.524) (drill 0.762) (layers "*.Cu" "*.Mask")
-      (net 6 "UART_0_TX") (pinfunction "Pin_2") (pintype "passive"))
+      (net 7 "UART_0_RX") (pinfunction "Pin_2") (pintype "passive"))
     (pad "3" thru_hole circle (at 1.27 0 90) (size 1.524 1.524) (drill 0.762) (layers "*.Cu" "*.Mask")
-      (net 7 "UART_0_RX") (pinfunction "Pin_3") (pintype "passive"))
+      (net 6 "UART_0_TX") (pinfunction "Pin_3") (pintype "passive"))
     (pad "4" thru_hole circle (at 3.81 0 90) (size 1.524 1.524) (drill 0.762) (layers "*.Cu" "*.Mask")
       (net 33 "Earth") (pinfunction "Pin_4") (pintype "passive"))
@@
   (segment (start 147.734 129.032) (end 146.563 129.032) (width 0.25) (layer "B.Cu") (net 5))
   (segment (start 146.563 129.032) (end 145.862 128.331) (width 0.25) (layer "B.Cu") (net 5))
-  (segment (start 135.067 92.39) (end 135.067 91.31237) (width 0.25) (layer "F.Cu") (net 6))
-  (segment (start 138.68837 87.691) (end 141.136 87.691) (width 0.25) (layer "F.Cu") (net 6))
-  (segment (start 135.067 91.31237) (end 138.68837 87.691) (width 0.25) (layer "F.Cu") (net 6))
-  (segment (start 140.501 89.596) (end 141.136 90.231) (width 0.25) (layer "B.Cu") (net 7))
-  (segment (start 135.067 89.596) (end 140.501 89.596) (width 0.25) (layer "B.Cu") (net 7))
+  (segment (start 135.067 89.596) (end 139.231 89.596) (width 0.25) (layer "B.Cu") (net 6))
+  (segment (start 139.231 89.596) (end 141.136 87.691) (width 0.25) (layer "B.Cu") (net 6))
+  (segment (start 135.067 92.39) (end 137.226 90.231) (width 0.25) (layer "F.Cu") (net 7))
+  (segment (start 137.226 90.231) (end 141.136 90.231) (width 0.25) (layer "F.Cu") (net 7))
   (segment (start 150.071 132.096) (end 158.916 123.251) (width 0.25) (layer "F.Cu") (net 10))
   (segment (start 135.53 132.096) (end 150.071 132.096) (width 0.25) (layer "F.Cu") (net 10))

Commit message: Transistor footprint correction - BC817
Replaced generic transistor symbol with the BC817 in a SOT23 package.
Fixed footprint allocation and re-done PCB traces to accomodate change.
Parts:
- Q1, Q2: value NPN -> BC817
- moved Q1 0.75 mm to (144.5, 122.9)
- moved Q2 0.42 mm to (144.5, 127.4)
Connections:
- Q1 pad 1: Net-(Q1-C) -> Net-(Q1-B)
- Q1 pad 2: Net-(Q1-B) -> SCL
- Q1 pad 3: SCL -> Net-(Q1-C)
- Q2 pad 1: Net-(Q2-C) -> Net-(Q2-B)
- Q2 pad 2: Net-(Q2-B) -> SCL
- Q2 pad 3: SCL -> Net-(Q2-C)
Routing:
- net SCL: track 20.7 -> 22.9 mm, vias 0 -> 3
- net Net-(Q1-C): track 14.8 -> 12.6 mm
- net Net-(Q1-B): track 4.02 -> 5.48 mm
- net Net-(Q2-B): track 2.16 -> 3.57 mm
- net Net-(Q2-C): track 20.3 -> 19.0 mm
Changed lines of the file:
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@@
       (drillshape 0)
       (scaleselection 1)
-      (outputdirectory "Gerber_Output/")
+      (outputdirectory "LiDAR_Breakout_Board/")
     )
   )
@@
   )
   (footprint "Package_TO_SOT_SMD:SOT-23" (layer "B.Cu")
-    (at 144.9245 122.301 180)
+    (at 144.5029 122.9158 180)
     (descr "SOT, 3 Pin (https://www.jedec.org/system/files/docs/to-236h.pdf variant AB), generated with kicad-footprint-generator ipc_gullwing_generator.py")
     (tags "SOT TO_SOT_SMD")
     (property "Sheetfile" "LiDAR-Board.kicad_sch")
     (property "Sheetname" "")
-    (property "Sim.Device" "NPN")
-    (property "Sim.Pins" "1=C 2=B 3=E")
-    (property "Sim.Type" "GUMMELPOON")
-    (property "ki_description" "Bipolar transistor symbol for simulation only, substrate tied to the emitter")
-    (property "ki_keywords" "simulation")
+    (property "ki_description" "0.8A Ic, 45V Vce, NPN Transistor, SOT-23")
+    (property "ki_keywords" "NPN Transistor")
     (attr smd)
     (fp_text reference "Q1" (at 0 2.4) (layer "B.SilkS")
         (effects (font (size 1 1) (thickness 0.15)) (justify mirror))
     )
-    (fp_text value "NPN" (at 0 -2.4) (layer "B.Fab")
+    (fp_text value "BC817" (at 0 -2.4) (layer "B.Fab")
         (effects (font (size 1 1) (thickness 0.15)) (justify mirror))
     )
+    (fp_text user "${REFERENCE}" (at 0 0) (layer "B.Fab")
+        (effects (font (size 0.32 0.32) (thickness 0.05)) (justify mirror))
+    )
     (fp_line (start 0 -1.56) (end -0.65 -1.56)
       (stroke (width 0.12) (type solid)) (layer "B.SilkS"))
@@
       (stroke (width 0.1) (type solid)) (layer "B.Fab"))
     (pad "1" smd roundrect (at -0.9375 0.95 180) (size 1.475 0.6) (layers "B.Cu" "B.Paste" "B.Mask") (roundrect_rratio 0.25)
-      (net 1 "Net-(Q1-C)") (pinfunction "C") (pintype "open_collector"))
+      (net 2 "Net-(Q1-B)") (pinfunction "B") (pintype "input"))
     (pad "2" smd roundrect (at -0.9375 -0.95 180) (size 1.475 0.6) (layers "B.Cu" "B.Paste" "B.Mask") (roundrect_rratio 0.25)
-      (net 2 "Net-(Q1-B)") (pinfunction "B") (pintype "input"))
+      (net 3 "SCL") (pinfunction "E") (pintype "passive"))
     (pad "3" smd roundrect (at 0.9375 0 180) (size 1.475 0.6) (layers "B.Cu" "B.Paste" "B.Mask") (roundrect_rratio 0.25)
-      (net 3 "SCL") (pinfunction "E") (pintype "open_emitter"))
+      (net 1 "Net-(Q1-C)") (pinfunction "C") (pintype "passive"))
     (model "${KICAD6_3DMODEL_DIR}/Package_TO_SOT_SMD.3dshapes/SOT-23.wrl"
       (offset (xyz 0 0 0))
@@
   )
   (footprint "Package_TO_SOT_SMD:SOT-23" (layer "B.Cu")
-    (at 144.9245 127.381 180)
+    (at 144.5029 127.3658 180)
     (descr "SOT, 3 Pin (https://www.jedec.org/system/files/docs/to-236h.pdf variant AB), generated with kicad-footprint-generator ipc_gullwing_generator.py")
     (tags "SOT TO_SOT_SMD")
     (property "Sheetfile" "LiDAR-Board.kicad_sch")
     (property "Sheetname" "")
-    (property "Sim.Device" "NPN")
-    (property "Sim.Pins" "1=C 2=B 3=E")
-    (property "Sim.Type" "GUMMELPOON")
-    (property "ki_description" "Bipolar transistor symbol for simulation only, substrate tied to the emitter")
-    (property "ki_keywords" "simulation")
+    (property "ki_description" "0.8A Ic, 45V Vce, NPN Transistor, SOT-23")
+    (property "ki_keywords" "NPN Transistor")
     (attr smd)
-    (fp_text reference "Q2" (at -0.0485 -3.744) (layer "B.SilkS")
+    (fp_text reference "Q2" (at 0.4849 -2.5552) (layer "B.SilkS")
         (effects (font (size 1 1) (thickness 0.15)) (justify mirror))
     )
-    (fp_text value "NPN" (at 0 -2.4) (layer "B.Fab")
+    (fp_text value "BC817" (at 0 -2.4) (layer "B.Fab")
         (effects (font (size 1 1) (thickness 0.15)) (justify mirror))
     )
@@
       (stroke (width 0.1) (type solid)) (layer "B.Fab"))
     (pad "1" smd roundrect (at -0.9375 0.95 180) (size 1.475 0.6) (layers "B.Cu" "B.Paste" "B.Mask") (roundrect_rratio 0.25)
-      (net 4 "Net-(Q2-C)") (pinfunction "C") (pintype "open_collector"))
+      (net 5 "Net-(Q2-B)") (pinfunction "B") (pintype "input"))
     (pad "2" smd roundrect (at -0.9375 -0.95 180) (size 1.475 0.6) (layers "B.Cu" "B.Paste" "B.Mask") (roundrect_rratio 0.25)
-      (net 5 "Net-(Q2-B)") (pinfunction "B") (pintype "input"))
+      (net 3 "SCL") (pinfunction "E") (pintype "passive"))
     (pad "3" smd roundrect (at 0.9375 0 180) (size 1.475 0.6) (layers "B.Cu" "B.Paste" "B.Mask") (roundrect_rratio 0.25)
-      (net 3 "SCL") (pinfunction "E") (pintype "open_emitter"))
+      (net 4 "Net-(Q2-C)") (pinfunction "C") (pintype "passive"))
     (model "${KICAD6_3DMODEL_DIR}/Package_TO_SOT_SMD.3dshapes/SOT-23.wrl"
       (offset (xyz 0 0 0))
@@
     (effects (font (size 1.5 1.5) (thickness 0.3) bold) (justify left bottom mirror))
   )
-  (segment (start 145.862 121.351) (end 142.301 121.351) (width 0.25) (layer "B.Cu") (net 1))
-  (segment (start 136.077 127.829) (end 134.94 128.966) (width 0.25) (layer "B.Cu") (net 1))
-  (segment (start 136.077 126.553) (end 136.077 127.829) (width 0.25) (layer "B.Cu") (net 1))
-  (segment (start 142.301 121.351) (end 141.626 122.026) (width 0.25) (layer "B.Cu") (net 1))
-  (segment (start 141.626 122.026) (end 140.604 122.026) (width 0.25) (layer "B.Cu") (net 1))
-  (segment (start 140.604 122.026) (end 136.077 126.553) (width 0.25) (layer "B.Cu") (net 1))
-  (segment (start 147.734 125.123) (end 147.734 126.492) (width 0.25) (layer "B.Cu") (net 2))
-  (segment (start 145.862 123.251) (end 147.734 125.123) (width 0.25) (layer "B.Cu") (net 2))
+  (segment (start 136.077 126.553) (end 140.604 122.026) (width 0.25) (layer "B.Cu") (net 1))
+  (segment (start 140.604 122.026) (end 142.6756 122.026) (width 0.25) (layer "B.Cu") (net 1))
+  (segment (start 142.6756 122.026) (end 143.5654 122.9158) (width 0.25) (layer "B.Cu") (net 1))
+  (segment (start 134.94 128.966) (end 136.077 127.829) (width 0.25) (layer "B.Cu") (net 1))
+  (segment (start 136.077 127.829) (end 136.077 126.553) (width 0.25) (layer "B.Cu") (net 1))
+  (segment (start 145.4404 121.9658) (end 147.734 124.2594) (width 0.25) (layer "B.Cu") (net 2))
+  (segment (start 147.734 124.2594) (end 147.734 126.492) (width 0.25) (layer "B.Cu") (net 2))
+  (segment (start 145.4404 129.6924) (end 146.4056 129.6924) (width 0.25) (layer "F.Cu") (net 3))
+  (segment (start 146.558 129.54) (end 146.558 125.222) (width 0.25) (layer "F.Cu") (net 3))
+  (segment (start 146.4056 129.6924) (end 146.558 129.54) (width 0.25) (layer "F.Cu") (net 3))
+  (segment (start 149.352 125.222) (end 150.622 123.952) (width 0.25) (layer "F.Cu") (net 3))
+  (segment (start 146.558 125.222) (end 149.352 125.222) (width 0.25) (layer "F.Cu") (net 3))
+  (via (at 145.4404 129.6924) (size 0.8) (drill 0.4) (layers "F.Cu" "B.Cu") (net 3))
+  (via (at 150.622 123.952) (size 0.8) (drill 0.4) (layers "F.Cu" "B.Cu") (net 3))
+  (via (at 146.558 125.222) (size 0.8) (drill 0.4) (layers "F.Cu" "B.Cu") (net 3))
+  (segment (start 145.4404 129.6924) (end 145.4404 128.3158) (width 0.25) (layer "B.Cu") (net 3))
+  (segment (start 150.622 123.952) (end 154.051 123.952) (width 0.25) (layer "B.Cu") (net 3))
+  (segment (start 146.558 124.9834) (end 145.4404 123.8658) (width 0.25) (layer "B.Cu") (net 3))
+  (segment (start 146.558 125.222) (end 146.558 124.9834) (width 0.25) (layer "B.Cu") (net 3))
   (segment (start 157.292 120.711) (end 158.916 120.711) (width 0.25) (layer "B.Cu") (net 3))
-  (segment (start 143.987 122.301) (end 143.987 127.381) (width 0.25) (layer "B.Cu") (net 3))
-  (segment (start 155.702 122.301) (end 157.292 120.711) (width 0.25) (layer "B.Cu") (net 3))
-  (segment (start 143.987 122.301) (end 155.702 122.301) (width 0.25) (layer "B.Cu") (net 3))
-  (segment (start 145.481 124.775) (end 145.481 117.526) (width 0.25) (layer "F.Cu") (net 4))
+  (segment (start 154.051 123.952) (end 157.292 120.711) (width 0.25) (layer "B.Cu") (net 3))
+  (segment (start 143.256 125.222) (end 143.256 117.491) (width 0.25) (layer "F.Cu") (net 4))
+  (segment (start 142.621 116.856) (end 135.911 116.856) (width 0.25) (layer "F.Cu") (net 4))
   (segment (start 135.911 116.856) (end 134.94 115.885) (width 0.25) (layer "F.Cu") (net 4))
-  (segment (start 145.481 117.526) (end 144.811 116.856) (width 0.25) (layer "F.Cu") (net 4))
-  (segment (start 144.811 116.856) (end 135.911 116.856) (width 0.25) (layer "F.Cu") (net 4))
-  (via (at 145.481 124.775) (size 0.8) (drill 0.4) (layers "F.Cu" "B.Cu") (net 4))
-  (segment (start 145.862 126.431) (end 145.862 125.156) (width 0.25) (layer "B.Cu") (net 4))
-  (segment (start 145.862 125.156) (end 145.481 124.775) (width 0.25) (layer "B.Cu") (net 4))
-  (segment (start 147.734 129.032) (end 146.563 129.032) (width 0.25) (layer "B.Cu") (net 5))
-  (segment (start 146.563 129.032) (end 145.862 128.331) (width 0.25) (layer "B.Cu") (net 5))
+  (segment (start 143.256 117.491) (end 142.621 116.856) (width 0.25) (layer "F.Cu") (net 4))
+  (via (at 143.256 125.222) (size 0.8) (drill 0.4) (layers "F.Cu" "B.Cu") (net 4))
+  (segment (start 143.5654 125.5314) (end 143.256 125.222) (width 0.25) (layer "B.Cu") (net 4))
+  (segment (start 143.5654 127.3658) (end 143.5654 125.5314) (width 0.25) (layer "B.Cu") (net 4))
+  (segment (start 145.4404 126.7384) (end 147.734 129.032) (width 0.25) (layer "B.Cu") (net 5))
+  (segment (start 145.4404 126.4158) (end 145.4404 126.7384) (width 0.25) (layer "B.Cu") (net 5))
   (segment (start 135.067 89.596) (end 139.231 89.596) (width 0.25) (layer "B.Cu") (net 6))
   (segment (start 139.231 89.596) (end 141.136 87.691) (width 0.25) (layer "B.Cu") (net 6))
