File: LiDAR-Main/Schematic/LiDAR-Board/LiDAR-Board.kicad_sch (KiCad schematic)
At the start: 8 parts, among them Q1 NPN, Q2 NPN, U1 Pico

Commit message: Schematic update pre-footprint
Parts:
- U1: footprint RPi_Pico:RPi_Pico_SMD_TH -> HEVCS_Sensor_Footprints:Pi_Pico; symbol MCU_RaspberryPi_and_Boards:Pico -> HEVCS_Sensors:Pico
Connections:
- net IMU SCL is gone; now on net IMU_SCL: U1.9 (GPIO6)
- net IMU SDA is gone; now on net IMU_SDA: U1.10 (GPIO7)
- no-connect marks 3 -> 32
Changed lines of the file:
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@@
   (junction (at 182.245 72.39) (diameter 0) (color 0 0 0 0)
   )
+  (no_connect (at 93.98 114.935))
+  (no_connect (at 93.98 122.555))
+  (no_connect (at 58.42 81.915))
+  (no_connect (at 93.98 89.535))
   (no_connect (at 196.85 80.01))
+  (no_connect (at 93.98 120.015))
+  (no_connect (at 93.98 102.235))
+  (no_connect (at 93.98 94.615))
+  (no_connect (at 93.98 99.695))
+  (no_connect (at 58.42 104.775))
+  (no_connect (at 93.98 97.155))
+  (no_connect (at 93.98 74.295))
+  (no_connect (at 58.42 109.855))
+  (no_connect (at 93.98 86.995))
+  (no_connect (at 58.42 107.315))
+  (no_connect (at 93.98 117.475))
   (no_connect (at 196.85 85.09))
+  (no_connect (at 78.74 127.635))
+  (no_connect (at 93.98 104.775))
+  (no_connect (at 58.42 99.695))
+  (no_connect (at 58.42 112.395))
+  (no_connect (at 58.42 92.075))
+  (no_connect (at 93.98 112.395))
+  (no_connect (at 76.2 127.635))
+  (no_connect (at 73.66 127.635))
+  (no_connect (at 58.42 102.235))
+  (no_connect (at 58.42 114.935))
+  (no_connect (at 58.42 79.375))
   (no_connect (at 196.85 82.55))
+  (no_connect (at 58.42 84.455))
+  (no_connect (at 93.98 92.075))
+  (no_connect (at 93.98 81.915))
   (wire (pts (xy 137.795 67.31) (xy 193.675 67.31))
     (stroke (width 0) (type default))
@@
     )
   )
-  (global_label "IMU SDA" (shape bidirectional) (at 58.42 97.155 180) (fields_autoplaced)
-    (effects (font (size 1.27 1.27)) (justify right))
-    (property "Intersheetrefs" "${INTERSHEET_REFS}" (at 46.6861 97.155 0)
+  (global_label "IMU_SDA" (shape bidirectional) (at 58.42 97.155 180) (fields_autoplaced)
+    (effects (font (size 1.27 1.27)) (justify right))
+    (property "Intersheetrefs" "${INTERSHEET_REFS}" (at 46.4805 97.155 0)
       (effects (font (size 1.27 1.27)) (justify right) hide)
     )
@@
     )
   )
-  (global_label "IMU SCL" (shape output) (at 58.42 94.615 180) (fields_autoplaced)
-    (effects (font (size 1.27 1.27)) (justify right))
-    (property "Intersheetrefs" "${INTERSHEET_REFS}" (at 47.8579 94.615 0)
+  (global_label "IMU_SCL" (shape output) (at 58.42 94.615 180) (fields_autoplaced)
+    (effects (font (size 1.27 1.27)) (justify right))
+    (property "Intersheetrefs" "${INTERSHEET_REFS}" (at 47.6523 94.615 0)
       (effects (font (size 1.27 1.27)) (justify right) hide)
     )
@@
     )
   )
-  (symbol (lib_id "MCU_RaspberryPi_and_Boards:Pico") (at 76.2 98.425 0) (unit 1)
+  (symbol (lib_id "HEVCS_Sensors:Pico") (at 76.2 98.425 0) (unit 1)
     (in_bom yes) (on_board yes) (dnp no) (fields_autoplaced)
     (property "Reference" "U1" (at 76.2 68.58 0)
@@
       (effects (font (size 1.27 1.27)))
     )
-    (property "Footprint" "RPi_Pico:RPi_Pico_SMD_TH" (at 76.2 98.425 90)
-      (effects (font (size 1.27 1.27)) hide)
-    )
+    (property "Footprint" "HEVCS_Sensor_Footprints:Pi_Pico" (at 76.2 98.425 90)
+      (effects (font (size 1.27 1.27)) hide)
+    )

Commit message: Footprint Allocations
Parts:
- Q1, Q2: footprint (none) -> Package_TO_SOT_SMD:SOT-23
- R1, R2: footprint (none) -> Resistor_SMD:R_0603_1608Metric
- U2, U3, U4: footprint (none) -> HEVCS_Sensor_Footprints:Conn_01x05_MOLEX
Other:
- note added: "I2C Port 1"
Changed lines of the file:
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@@
     (stroke (width 0) (type default))
+  )
+  (text "I2C Port 1\n" (at 38.1 95.25 0)
+    (effects (font (size 1.27 1.27)) (justify left bottom))
   )
   (text "I2C Port 0\n" (at 41.91 88.265 0)
@@
       (effects (font (size 1.27 1.27)) (justify left))
     )
-    (property "Footprint" "" (at 198.755 59.69 0)
+    (property "Footprint" "Package_TO_SOT_SMD:SOT-23" (at 198.755 59.69 0)
       (effects (font (size 1.27 1.27)) hide)
     )
@@
       (effects (font (size 1.27 1.27)) (justify left))
     )
-    (property "Footprint" "" (at 198.755 73.025 0)
+    (property "Footprint" "Package_TO_SOT_SMD:SOT-23" (at 198.755 73.025 0)
       (effects (font (size 1.27 1.27)) hide)
     )
@@
       (effects (font (size 1.27 1.27)))
     )
-    (property "Footprint" "" (at 203.835 59.69 0)
+    (property "Footprint" "HEVCS_Sensor_Footprints:Conn_01x05_MOLEX" (at 203.835 59.69 0)
       (effects (font (size 1.27 1.27)) hide)
     )
@@
       (effects (font (size 1.27 1.27)))
     )
-    (property "Footprint" "" (at 126.365 74.803 90)
+    (property "Footprint" "Resistor_SMD:R_0603_1608Metric" (at 126.365 74.803 90)
       (effects (font (size 1.27 1.27)) hide)
     )
@@
       (effects (font (size 1.27 1.27)))
     )
-    (property "Footprint" "" (at 209.55 99.06 0)
+    (property "Footprint" "HEVCS_Sensor_Footprints:Conn_01x05_MOLEX" (at 209.55 99.06 0)
       (effects (font (size 1.27 1.27)) hide)
     )
@@
       (effects (font (size 1.27 1.27)))
     )
-    (property "Footprint" "" (at 203.835 46.355 0)
+    (property "Footprint" "HEVCS_Sensor_Footprints:Conn_01x05_MOLEX" (at 203.835 46.355 0)
       (effects (font (size 1.27 1.27)) hide)
     )
@@
       (effects (font (size 1.27 1.27)))
     )
-    (property "Footprint" "" (at 126.365 61.468 90)
-      (effects (font (size 1.27 1.27)) hide)
-    )
+    (property "Footprint" "Resistor_SMD:R_0603_1608Metric" (at 126.365 61.468 90)
+      (effects (font (size 1.27 1.27)) hide)
+    )

Commit message: Connector on schematic
Parts:
- added J1: Conn_01x04, symbol Connector_Generic:Conn_01x04
Connections:
- net Earth: now also J1.4 (Pin_4)
- net UART_0_RX: now also J1.3 (Pin_3)
- net UART_0_TX: now also J1.2 (Pin_2)
- net +5V renamed 5V_MAIN_BOARD
- net 5V_MAIN_BOARD: now also J1.1 (Pin_1)
Other:
- note added: "CONNECTOR FROM MAIN BOARD"
Changed lines of the file:
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@@
+    (stroke (width 0) (type default))
+  )
+  (wire (pts (xy 101.6 57.15) (xy 101.6 76.835))
     (stroke (width 0) (type default))
   )
@@
     (stroke (width 0) (type default))
   )
-  (wire (pts (xy 101.6 63.5) (xy 101.6 76.835))
-    (stroke (width 0) (type default))
-  )
   (wire (pts (xy 177.8 72.39) (xy 177.8 95.25))
     (stroke (width 0) (type default))
@@
     (stroke (width 0) (type default))
   )
+  (wire (pts (xy 31.115 58.42) (xy 37.465 58.42))
+    (stroke (width 0) (type default))
+  )
   (wire (pts (xy 101.6 76.835) (xy 93.98 76.835))
     (stroke (width 0) (type default))
@@
     (stroke (width 0) (type default))
   )
+  (wire (pts (xy 37.465 58.42) (xy 37.465 61.595))
+    (stroke (width 0) (type default))
+  )
   (wire (pts (xy 93.98 79.375) (xy 101.6 79.375))
     (stroke (width 0) (type default))
@@
   (wire (pts (xy 182.245 72.39) (xy 193.675 72.39))
     (stroke (width 0) (type default))
+  )
+  (text "CONNECTOR FROM MAIN BOARD\n" (at 42.545 60.325 0)
+    (effects (font (size 1.27 1.27)) (justify left bottom))
   )
   (text "I2C Port 1\n" (at 38.1 95.25 0)
@@
     )
   )
+  (global_label "UART_0_RX" (shape output) (at 31.115 55.88 0) (fields_autoplaced)
+    (effects (font (size 1.27 1.27)) (justify left))
+    (property "Intersheetrefs" "${INTERSHEET_REFS}" (at 44.3017 55.88 0)
+      (effects (font (size 1.27 1.27)) (justify left) hide)
+    )
+  )
+  (global_label "5V_MAIN_BOARD" (shape input) (at 101.6 57.15 0) (fields_autoplaced)
+    (effects (font (size 1.27 1.27)) (justify left))
+    (property "Intersheetrefs" "${INTERSHEET_REFS}" (at 119.4435 57.15 0)
+      (effects (font (size 1.27 1.27)) (justify left) hide)
+    )
+  )
   (global_label "SDA" (shape bidirectional) (at 58.42 89.535 180) (fields_autoplaced)
     (effects (font (size 1.27 1.27)) (justify right))
@@
     )
   )
+  (global_label "5V_MAIN_BOARD" (shape input) (at 177.8 72.39 180) (fields_autoplaced)
+    (effects (font (size 1.27 1.27)) (justify right))
+    (property "Intersheetrefs" "${INTERSHEET_REFS}" (at 159.9565 72.39 0)
+      (effects (font (size 1.27 1.27)) (justify right) hide)
+    )
+  )
+  (global_label "UART_0_TX" (shape input) (at 31.115 53.34 0) (fields_autoplaced)
+    (effects (font (size 1.27 1.27)) (justify left))
+    (property "Intersheetrefs" "${INTERSHEET_REFS}" (at 43.9993 53.34 0)
+      (effects (font (size 1.27 1.27)) (justify left) hide)
+    )
+  )
   (global_label "IMU_SCL" (shape output) (at 58.42 94.615 180) (fields_autoplaced)
     (effects (font (size 1.27 1.27)) (justify right))
     (property "Intersheetrefs" "${INTERSHEET_REFS}" (at 47.6523 94.615 0)
       (effects (font (size 1.27 1.27)) (justify right) hide)
+    )
+  )
+  (global_label "5V_MAIN_BOARD" (shape output) (at 31.115 50.8 0) (fields_autoplaced)
+    (effects (font (size 1.27 1.27)) (justify left))
+    (property "Intersheetrefs" "${INTERSHEET_REFS}" (at 48.9585 50.8 0)
+      (effects (font (size 1.27 1.27)) (justify left) hide)
     )
   )
@@
         (path "/379f291a-31d3-4ed1-aaf1-b1b6ffabef49"
           (reference "U4") (unit 1)
+        )
+      )
+    )
+  )
+  (symbol (lib_id "power:Earth") (at 37.465 61.595 0) (unit 1)
+    (in_bom yes) (on_board yes) (dnp no) (fields_autoplaced)
+    (property "Reference" "#PWR01" (at 37.465 67.945 0)
+      (effects (font (size 1.27 1.27)) hide)
+    )
+    (property "Value" "Earth" (at 37.465 65.405 0)
+      (effects (font (size 1.27 1.27)) hide)
+    )
+    (property "Footprint" "" (at 37.465 61.595 0)
+      (effects (font (size 1.27 1.27)) hide)
+    )
+    (property "Datasheet" "~" (at 37.465 61.595 0)
+      (effects (font (size 1.27 1.27)) hide)
+    )
+    (pin "1")
+    (instances
+      (project "LiDAR-Board"
+        (path "/379f291a-31d3-4ed1-aaf1-b1b6ffabef49"
+          (reference "#PWR01") (unit 1)
         )
       )
@@
     )
   )
+  (symbol (lib_id "Connector_Generic:Conn_01x04") (at 26.035 53.34 0) (mirror y) (unit 1)
+    (in_bom yes) (on_board yes) (dnp no)
+    (property "Reference" "J1" (at 26.035 64.135 0)
+      (effects (font (size 1.27 1.27)))
+    )
+    (property "Value" "Conn_01x04" (at 26.035 61.595 0)
+      (effects (font (size 1.27 1.27)))
+    )
+    (property "Footprint" "" (at 26.035 53.34 0)
+      (effects (font (size 1.27 1.27)) hide)
+    )
+    (property "Datasheet" "~" (at 26.035 53.34 0)
+      (effects (font (size 1.27 1.27)) hide)
+    )
+    (pin "1")
+    (pin "2")
+    (pin "3")
+    (pin "4")
+    (instances
+      (project "LiDAR-Board"
+        (path "/379f291a-31d3-4ed1-aaf1-b1b6ffabef49"
+          (reference "J1") (unit 1)
+        )
+      )
+    )
+  )
   (symbol (lib_id "VL53L5CX_KiCAD:VL53L5CX_Pimoroni") (at 203.835 46.355 0) (mirror y) (unit 1)
     (in_bom yes) (on_board yes) (dnp no) (fields_autoplaced)
@@
         )
       )
-    )
-  )
-  (symbol (lib_id "power:+5V") (at 101.6 63.5 0) (unit 1)
-    (in_bom yes) (on_board yes) (dnp no) (fields_autoplaced)
-    (property "Reference" "#PWR02" (at 101.6 67.31 0)
-      (effects (font (size 1.27 1.27)) hide)
-    )
-    (property "Value" "+5V" (at 101.6 59.69 0)
-      (effects (font (size 1.27 1.27)))
-    )
-    (property "Footprint" "" (at 101.6 63.5 0)
-      (effects (font (size 1.27 1.27)) hide)
-    )
-    (property "Datasheet" "" (at 101.6 63.5 0)
-      (effects (font (size 1.27 1.27)) hide)
-    )
-    (pin "1")
-    (instances
-      (project "LiDAR-Board"
-        (path "/379f291a-31d3-4ed1-aaf1-b1b6ffabef49"
-          (reference "#PWR02") (unit 1)
-        )
-      )
-    )
-  )
-  (symbol (lib_id "power:+5V") (at 177.8 72.39 0) (unit 1)
-    (in_bom yes) (on_board yes) (dnp no) (fields_autoplaced)
-    (property "Reference" "#PWR01" (at 177.8 76.2 0)
-      (effects (font (size 1.27 1.27)) hide)
-    )
-    (property "Value" "+5V" (at 177.8 68.58 0)
-      (effects (font (size 1.27 1.27)))
-    )
-    (property "Footprint" "" (at 177.8 72.39 0)
-      (effects (font (size 1.27 1.27)) hide)
-    )
-    (property "Datasheet" "" (at 177.8 72.39 0)
-      (effects (font (size 1.27 1.27)) hide)
-    )
-    (pin "1")
-    (instances
-      (project "LiDAR-Board"
-        (path "/379f291a-31d3-4ed1-aaf1-b1b6ffabef49"
-          (reference "#PWR01") (unit 1)
-        )
-      )

Commit message: PCB Finished w/earths
Parts:
- J1: footprint (none) -> HEVCS_Sensor_Footprints:Conn_01x04_MOLEX
Connections:
- net Earth: now also U1.23 (GND), U1.3 (GND), U2.5 (GND), U3.5 (GND); no longer U2. (GND), U3. (GND)
- net IMU_INT: now also U1.17 (GPIO13); no longer U1.18 (GND)
- net INT_1: now also U1.22 (GPIO17); no longer U1.19 (GPIO14)
- net INT_2: now also U1.21 (GPIO16); no longer U1.20 (GPIO15)
- net SCL: now also U1.27 (GPIO21); no longer U1.6 (GPIO4)
- net SDA: now also U1.26 (GPIO20); no longer U1.7 (GPIO5)
- net at R2.1: now also U1.24 (GPIO18); no longer U1.26 (GPIO20)
- net at U1.25 (GPIO19): now also R1.1
- no-connect marks 32 -> 30
