File: BreakawayConnector/BreakawayConnector/BreakawayConnector.kicad_pcb (KiCad board)
At the start: 2 copper layers, 40 x 40 mm, 2 parts, among them J1 Conn_01x10, J2 Conn_01x10

Commit message: Added identifier
Other:
- board text added: "DC, LW, JP, NH"
- board text added: "HEVCS"
Changed lines of the file:
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@@
   (gr_circle (center 100 100) (end 120 100)
     (stroke (width 0.1) (type default)) (fill none) (layer "Edge.Cuts"))
+  (gr_text "DC, LW, JP, NH" (at 94.7 119.2) (layer "F.SilkS")
+    (effects (font (size 1 1) (thickness 0.1)) (justify left bottom))
+  )
+  (gr_text "HEVCS\n" (at 97.8 117.9) (layer "F.SilkS")
+    (effects (font (size 1 1) (thickness 0.1)) (justify left bottom))
+  )
   (segment (start 100 85) (end 100 87.5) (width 0.5) (layer "F.Cu") (net 1))
   (segment (start 92.6527 89.3342) (end 92.6527 89.8873) (width 0.5) (layer "F.Cu") (net 2))

Commit message: Added Gerber files for breakaway connector and controller.
Other:
- board text added: "DC, JP, LW, NH"
- board text removed: "DC, LW, JP, NH"
Changed lines of the file:
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@@
       (outputformat 1)
       (mirror false)
-      (drillshape 1)
+      (drillshape 0)
       (scaleselection 1)
-      (outputdirectory "")
+      (outputdirectory "Gerbers/")
     )
   )
@@
   (gr_circle (center 100 100) (end 120 100)
     (stroke (width 0.1) (type default)) (fill none) (layer "Edge.Cuts"))
-  (gr_text "DC, LW, JP, NH" (at 94.7 119.2) (layer "F.SilkS")
+  (gr_text "DC, JP, LW, NH" (at 94.7 119.2) (layer "F.SilkS")
     (effects (font (size 1 1) (thickness 0.1)) (justify left bottom))
   )
